File: nanoComp.kicad_pcb (KiCad board)
At the start: 2 copper layers, 90 x 70 mm, 21 parts, among them J1 USB_C_Receptacle_PowerOnly_6P, J2 USB_A, J3 USB_A, J4 Conn_01x06_Pin, J5 Conn_01x14, J6 Conn_01x04, SW1 SW_Wuerth_450301014042

Commit message: Finishing touches + manufacturing files
Parts:
- added REF**: OSHW-Logo2_9.8x8mm_SilkScreen, Symbol:OSHW-Logo2_9.8x8mm_SilkScreen, F.Cu at (162.5, 115.0)
- D1: value 1N5819WS -> 1N5819HW-7-F; footprint Diode_SMD:D_SOD-323_HandSoldering -> Diode_SMD:D_SOD-123
- moved D1 0.50 mm to (105.5, 76.0)
Routing:
- net Net-(D1-A): track 14.9 -> 14.0 mm
Other:
- board text added: "https://github.com/venomix666/nanoComp"
